Commit message: Self-collision detection

File: test/data/robot.urdf (robot description, URDF)
Before this commit: robot robot_arm, 8 links, 7 joints
Joints:
- joint joint1: limit lower=-1 upper=1 -> (none)
- joint joint2: limit lower=-1 -> (none)
- joint joint3: limit upper=1 -> (none)

Commit message: Fix self-collision detection

File: test/data/robot.urdf (robot description, URDF)
Before this commit: robot robot_arm, 8 links, 7 joints
Links:
- link link1: geometry collision cylinder length=0.11 radius=0.05
- link link2: geometry collision cylinder length=0.1 radius=0.05; collision cylinder length=0.18 radius=0.05
- link link4: geometry collision cylinder length=0.24 radius=0.05
- link link5: geometry collision cylinder length=0.1 radius=0.05; collision cylinder length=0.296 radius=0.05
